File: Hardware/Friend.sch (KiCad schematic (older format))
At the start: 9 parts

Commit message: reset, caps and power regulation
Parts:
- removed F?: FUSE, symbol FUSE
- added 18pF?: C, symbol C
- added P?: CONN_01X02, symbol CONN_01X02
- added R?: R, symbol R
- added SW?: SW_PUSH, symbol SW_PUSH
- added U?: LM2931AZ-3.3/5.0, TO92-123, symbol LM2931AZ-3.3/5.0
Connections:
- net labels added: VCC, VSS
- wire segments 26 -> 45
Changed lines of the file:
@@
 LIBS:contrib
 LIBS:valves
+LIBS:Friend-cache
 EELAYER 25 0
 EELAYER END
@@
 $EndComp
 $Comp
-L FUSE F?
-U 1 1 565C840E
-P 2900 2750
-F 0 "F?" H 3000 2800 50  0000 C CNN
-F 1 "FUSE" H 2800 2700 50  0000 C CNN
-F 2 "" H 2900 2750 60  0000 C CNN
-F 3 "" H 2900 2750 60  0000 C CNN
-	1    2900 2750
-	1    0    0    -1
-$EndComp
-$Comp
 L +5V #PWR?
 U 1 1 565C854B
@@
 	2600 3100 2600 2750
 Wire Wire Line
-	2600 2750 2650 2750
-Wire Wire Line
-	3150 2750 3350 2750
+	2600 2750 3350 2750
 Wire Wire Line
 	3250 2750 3250 2650
@@
 	2850 3950 2700 3950
 Wire Wire Line
-	4650 4700 4650 4800
-Wire Wire Line
-	4650 4800 3950 4800
+	4650 4800 4650 4700
+Wire Wire Line
+	3950 4800 4650 4800
 Wire Wire Line
 	4100 4700 4100 4800
@@
 	4550 4700 4550 4800
 Connection ~ 4550 4800
+$Comp
+L SW_PUSH SW?
+U 1 1 565CA2C4
+P 2850 1550
+F 0 "SW?" H 3000 1660 50  0000 C CNN
+F 1 "SW_PUSH" H 2850 1470 50  0000 C CNN
+F 2 "" H 2850 1550 60  0000 C CNN
+F 3 "" H 2850 1550 60  0000 C CNN
+	1    2850 1550
+	1    0    0    -1
+$EndComp
+$Comp
+L GND #PWR?
+U 1 1 565CA334
+P 2400 1550
+F 0 "#PWR?" H 2400 1300 50  0001 C CNN
+F 1 "GND" H 2400 1400 50  0000 C CNN
+F 2 "" H 2400 1550 60  0000 C CNN
+F 3 "" H 2400 1550 60  0000 C CNN
+	1    2400 1550
+	0    1    1    0
+$EndComp
+Wire Wire Line
+	2400 1550 2550 1550
+Wire Wire Line
+	3150 1550 3350 1550
+$Comp
+L C 18pF?
+U 1 1 565CA400
+P 2900 3300
+F 0 "18pF?" H 2925 3400 50  0000 L CNN
+F 1 "C" H 2925 3200 50  0000 L CNN
+F 2 "" H 2938 3150 30  0000 C CNN
+F 3 "" H 2900 3300 60  0000 C CNN
+	1    2900 3300
+	-1   0    0    1
+$EndComp
+$Comp
+L GND #PWR?
+U 1 1 565CA494
+P 2900 3500
+F 0 "#PWR?" H 2900 3250 50  0001 C CNN
+F 1 "GND" H 2900 3350 50  0000 C CNN
+F 2 "" H 2900 3500 60  0000 C CNN
+F 3 "" H 2900 3500 60  0000 C CNN
+	1    2900 3500
+	1    0    0    -1
+$EndComp
+Wire Wire Line
+	2900 3500 2900 3450
+$Comp
+L +5V #PWR?
+U 1 1 565CA557
+P 4050 1150
+F 0 "#PWR?" H 4050 1000 50  0001 C CNN
+F 1 "+5V" H 4050 1290 50  0000 C CNN
+F 2 "" H 4050 1150 60  0000 C CNN
+F 3 "" H 4050 1150 60  0000 C CNN
+	1    4050 1150
+	1    0    0    -1
+$EndComp
+$Comp
+L VCC #PWR?
+U 1 1 565CA582
+P 4300 1150
+F 0 "#PWR?" H 4300 1000 50  0001 C CNN
+F 1 "VCC" H 4300 1300 50  0000 C CNN
+F 2 "" H 4300 1150 60  0000 C CNN
+F 3 "" H 4300 1150 60  0000 C CNN
+	1    4300 1150
+	1    0    0    -1
+$EndComp
+Wire Wire Line
+	4050 1300 4050 1150
+Wire Wire Line
+	4300 1150 4300 1300
+Wire Wire Line
+	4400 1300 4400 1200
+Wire Wire Line
+	4300 1200 4750 1200
+Connection ~ 4300 1200
+Wire Wire Line
+	4650 1200 4650 1300
+Connection ~ 4400 1200
+Wire Wire Line
+	4750 1200 4750 1300
+Connection ~ 4650 1200
+$Comp
+L CONN_01X02 P?
+U 1 1 565CA872
+P 6650 1450
+F 0 "P?" H 6650 1600 50  0000 C CNN
+F 1 "CONN_01X02" V 6750 1450 50  0000 C CNN
+F 2 "" H 6650 1450 60  0000 C CNN
+F 3 "" H 6650 1450 60  0000 C CNN
+	1    6650 1450
+	1    0    0    -1
+$EndComp
+$Comp
+L GND #PWR?
+U 1 1 565CAA15
+P 6300 1550
+F 0 "#PWR?" H 6300 1300 50  0001 C CNN
+F 1 "GND" H 6300 1400 50  0000 C CNN
+F 2 "" H 6300 1550 60  0000 C CNN
+F 3 "" H 6300 1550 60  0000 C CNN
+	1    6300 1550
+	0    1    1    0
+$EndComp
+Wire Wire Line
+	6450 1400 6300 1400
+Wire Wire Line
+	6300 1400 6300 1350
+Wire Wire Line
+	6450 1500 6300 1500
+Wire Wire Line
+	6300 1500 6300 1550
+$Comp
+L GND #PWR?
+U 1 1 565CAC8A
+P 5750 3650
+F 0 "#PWR?" H 5750 3400 50  0001 C CNN
+F 1 "GND" H 5750 3500 50  0000 C CNN
+F 2 "" H 5750 3650 60  0000 C CNN
+F 3 "" H 5750 3650 60  0000 C CNN
+	1    5750 3650
+	0    -1   -1   0
+$EndComp
+Wire Wire Line
+	5600 3650 5750 3650
+$Comp
+L R R?
+U 1 1 565CAD1A
+P 3250 1350
+F 0 "R?" V 3330 1350 50  0000 C CNN
+F 1 "R" V 3250 1350 50  0000 C CNN
+F 2 "" V 3180 1350 30  0000 C CNN
+F 3 "" H 3250 1350 30  0000 C CNN
+	1    3250 1350
+	1    0    0    -1
+$EndComp
+$Comp
+L VCC #PWR?
+U 1 1 565CAD77
+P 3250 1150
+F 0 "#PWR?" H 3250 1000 50  0001 C CNN
+F 1 "VCC" H 3250 1300 50  0000 C CNN
+F 2 "" H 3250 1150 60  0000 C CNN
+F 3 "" H 3250 1150 60  0000 C CNN
+	1    3250 1150
+	1    0    0    -1
+$EndComp
+Wire Wire Line
+	3250 1500 3250 1550
+Connection ~ 3250 1550
+Wire Wire Line
+	3250 1150 3250 1200
+Wire Wire Line
+	2900 3150 3350 3150
+$Comp
+L VSS #PWR?
+U 1 1 565CB152
+P 6300 1350
+F 0 "#PWR?" H 6300 1200 50  0001 C CNN
+F 1 "VSS" H 6300 1500 50  0000 C CNN
+F 2 "" H 6300 1350 60  0000 C CNN
+F 3 "" H 6300 1350 60  0000 C CNN
+	1    6300 1350
+	0    -1   -1   0
+$EndComp
+$Comp
+L LM2931AZ-3.3/5.0 U?
+U 1 1 565CB3AB
+P 6400 2100
+F 0 "U?" H 6400 2350 40  0000 C CNN
+F 1 "LM2931AZ-3.3/5.0" H 6400 2300 40  0000 C CNN
+F 2 "TO92-123" H 6400 2200 35  0000 C CIN
+F 3 "" H 6400 2100 60  0000 C CNN
+	1    6400 2100
+	1    0    0    -1
+$EndComp
+$Comp
+L VSS #PWR?
+U 1 1 565CB57E
+P 5900 2050
+F 0 "#PWR?" H 5900 1900 50  0001 C CNN
+F 1 "VSS" H 5900 2200 50  0000 C CNN
+F 2 "" H 5900 2050 60  0000 C CNN
+F 3 "" H 5900 2050 60  0000 C CNN
+	1    5900 2050
+	0    -1   -1   0
+$EndComp
+$Comp
+L VCC #PWR?
+U 1 1 565CB5F1
+P 6900 2050
+F 0 "#PWR?" H 6900 1900 50  0001 C CNN
+F 1 "VCC" H 6900 2200 50  0000 C CNN
+F 2 "" H 6900 2050 60  0000 C CNN
+F 3 "" H 6900 2050 60  0000 C CNN
+	1    6900 2050
+	0    1    1    0
+$EndComp
+$Comp
+L GND #PWR?
+U 1 1 565CB66A
+P 6400 2450
+F 0 "#PWR?" H 6400 2200 50  0001 C CNN
+F 1 "GND" H 6400 2300 50  0000 C CNN
+F 2 "" H 6400 2450 60  0000 C CNN
+F 3 "" H 6400 2450 60  0000 C CNN
+	1    6400 2450
+	1    0    0    -1
+$EndComp
+Wire Wire Line
+	5900 2050 6000 2050
+Wire Wire Line
+	6800 2050 6900 2050
+Wire Wire Line
+	6400 2350 6400 2450
 $EndSCHEMATC

Commit message: mpu-6050
Parts:
- added 0.1uF (x2), 0.1uF?, 2.2nF: C, symbol C
- added 10kΩ (x2): R, symbol R
- added U?: MPU-6050, symbol MPU-6050
Connections:
- net GND: now also 0.1uF.1, 0.1uF.1, 0.1uF?.1, 2.2nF.1, U?.1 (CLKIN), U?.11 (FSYNC), U?.18 (GND), U?.9 (AD0); no longer U?.2 (GND), U?.33 ((~HWB~)PE2)
- net VCC: now also 0.1uF.2, 10kΩ.2, 10kΩ.2, U?.13 (VDD)
- new net: 0.1uF.2, U?.10 (REGOUT)
- new net: 2.2nF.2, U?.20 (CPOUT)
- new net: 0.1uF?.2, U?.8 (VLOGIC)
- new net SCL: 10kΩ.1, U?.23 (SCL)
- new net SDA: 10kΩ.1, U?.24 (SDA)

Commit message: eprom for data storage
Parts:
- removed 10kΩ (x2): R, symbol R
- added 4.7kΩ (x2): R, symbol R
- added IC?: AT24CS64-SSHM, SO8, symbol AT24CS64-SSHM
Connections:
- net GND: now also U?.2 (GND), IC?.1 (A0), IC?.2 (A1), IC?.3 (A2), IC?.4 (GND), IC?.7 (WP)
- net SCL: now also U?.18 ((OC0B/SCL/INT0)PD0), 4.7kΩ.1, IC?.6 (SCL)
- net SDA: now also U?.19 ((SDA/INT1)PD1), 4.7kΩ.1, IC?.5 (SDA)
- net VCC: now also 4.7kΩ.2, 4.7kΩ.2, IC?.8 (VCC)
Other:
- moved on the sheet: U?

Commit message: dual ignition systems
one for good luck
Parts:
- added 10kΩ (x2): R, symbol R
- added P? (x2): CONN_01X02, symbol CONN_01X02
- added Q? (x2): FDS6890A, SO-8, symbol FDS6890A
Connections:
- net GND: now also 10kΩ.2, 10kΩ.2, Q?.1 (S), Q?.3 (S)
- net VSS: now also P?.1 (P1), P?.2 (P2)
- new net IGNd1: 10kΩ.1, 10kΩ.1, Q?.2 (G), Q?.4 (G)
- new net IGNo1: P?.1 (P1), Q?.7, Q?.8 (D)
- new net IGNo2: P?.2 (P2), Q?.5 (D), Q?.6
Other:
- moved on the sheet: IC?

Commit message: barometer
Parts:
- added 0.1uF (x2), 1uF: C, symbol C
- added 10uF: CP, symbol CP
- added U?: MPL3115A2, symbol MPL3115A2
Connections:
- net GND: now also 0.1uF.1, 0.1uF.2, 10uF.2, 1uF.1, U?.3 (GND)
- net SCL: now also U?.8 (SCL)
- net SDA: now also U?.7 (SDA)
- net VCC: now also 0.1uF.2, 10uF.1, 1uF.2, U?.1 (VDD), U?.4 (VDDIO)
- new net: 0.1uF.1, U?.2 (CAP)
